Commit message: urdf模型tf求解建立

File: ur_description/urdf/my_ur5_copy.urdf (robot description, URDF)
Before this commit: robot ur5, 15 links, 14 joints
Links:
- removed link world_link
Joints:
- removed joint base_world_joint
- joint base_support_joint_L: origin xyz=0.0 0.0 0.0 rpy=-0.61548 -2.61799 0.955316 -> xyz=0.0 0.25 0.0 rpy=-2.3562 0.0 0.0; parent world_link -> base_support_box_link

File: ur_description/urdf/my_ur5_joint_limited_robot.urdf.xacro (robot description, xacro)
@@ -63,4 +63,6 @@
       </collision>
     </link>
+  <link name="world_link" >
+  </link>
   <joint name="world_joint" type="fixed">
     <parent link="world" />
@@ -78,8 +80,13 @@
     <origin xyz="0.0 0.0 0.25" rpy="0.0 0.0 0.0" />
   </joint>
-   <joint name="base_support_joint_L" type="fixed">
+  <joint name="base_world_joint" type="fixed">
       <parent link="base_support_box_link" />
+      <child link = "world_link" />
+      <origin xyz="0.0 0.25 0.0" rpy="0.0 0.0 -1.5708" />
+  </joint>
+  <joint name="base_support_joint_L" type="fixed">
+      <parent link="world_link" />
       <child link = "base_link" />
-      <origin xyz="0.0 0.25 0.0" rpy="-2.3562 0.0 0.0" />
-    </joint>
+      <origin xyz="0.0 0.0 0.0" rpy="-0.61548 -2.61799 0.955316" />
+  </joint>
 </robot>
